Commit message: gatlin shows up in gazebo, but arm is not moving correctly

File: robots/gatlin_with_arm_and_head.urdf.xacro (robot description, xacro)
@@ -1,4 +1,5 @@
 <?xml version="1.0"?>
-<robot name="gatlin_robot" xmlns:xacro="http://ros.org/wiki/xacro">
+<robot name="turtlebot" xmlns:xacro="http://ros.org/wiki/xacro">
+<!-- <robot name="gatlin_robot" xmlns:xacro="http://ros.org/wiki/xacro"> -->
    <xacro:property name="PI" value="3.1415"/>
    <!-- Define a number of dimensions using properties -->
@@ -23,5 +24,5 @@
    <xacro:property name="wrist_llimit" value="-1.72"/>
    <xacro:property name="wrist_ulimit" value="1.68"/>
-   <xacro:include filename="$(find gatlin)/urdf/turtlebot_arm.xacro"/>
+   <xacro:include filename="$(find gatlin)/urdf/pincher_arm.urdf"/>
    <xacro:include filename="$(find gatlin)/urdf/pan_tilt_head.urdf.xacro" />
    <!-- Now we can start using the macros included above to define the actual robot -->
@@ -29,12 +30,14 @@
    <create/>
    <!-- Attach the stacks -->
+   <!-- <stack_circles parent="base_link"/> -->
    <stack_squares parent="base_link" offset="${stacks_offset}" top_plate="${top_plate}"/>
    <!-- Attach the pan and tilt head -->
+   <!-- <sensor_kinect  parent="base_link"/> -->
    <head name="head_base" parent="plate_3" color="White">
       <origin xyz="${head_offset_x} ${head_offset_y} ${head_offset_z}" rpy="${PI/2} 0 ${PI/2+head_offset_rotz}" />
    </head>
    <!-- Attach the arm -->
-   <turtlebot_arm parent="base_link" color="Gray" gripper_color="Gray" pincher_gripper="true" turtlebot_gripper="false">
-     <origin xyz="${arm_offset_x} ${arm_offset_y} ${arm_offset_z}" rpy="0 0 0" />
-   </turtlebot_arm>
+   <!-- <turtlebot_arm parent="base_link" color="Gray" gripper_color="Gray" pincher_gripper="true" turtlebot_gripper="false">
+      <origin xyz="${arm_offset_x} ${arm_offset_y} ${arm_offset_z}" rpy="0 0 0" />
+   </turtlebot_arm> -->
 </robot>

File: urdf/common_properties.urdf.xacro (robot description, xacro)
@@ -35,9 +35,9 @@
     </material>
   </xacro:property>
-  <xacro:property name="material_green">
+  <!-- <xacro:property name="material_green">
     <material name="green">
       <color rgba="0.0 0.8 0.0 1"/>
     </material>
-  </xacro:property>
+  </xacro:property> -->
   <xacro:property name="material_blue">
     <material name="blue">

File: urdf/create.urdf.xacro (robot description, xacro)
@@ -35,5 +35,5 @@
 	      <origin xyz=" 0 0 0.0308" rpy="0 0 0" />
 	      <geometry>
-	        <mesh filename="package://create_description/meshes/create_body.dae"/>
+	        <mesh filename="package://gatlin/meshes/create_body.dae"/>
 	      </geometry>
 	    </visual>

File: urdf/stacks/circles.urdf.xacro (robot description, xacro)
@@ -18,5 +18,5 @@
         <origin xyz=" 0 0 0 " rpy="0 0 0" />
         <geometry>
-          <mesh filename="package://gatlin/meshes/stacks/circles/68-02403-125_Spacer.dae"/>
+          <mesh filename="package://turtlebot_description/meshes/stacks/circles/68-02403-125_Spacer.dae"/>
         </geometry>
       </visual>
@@ -46,5 +46,5 @@
         <origin xyz=" 0 0 0 " rpy="0 0 0" />
         <geometry>
-          <mesh filename="package://gatlin/meshes/stacks/circles/68-04552-1000-RA_Turtlebot_M-F_Standoff.dae"/>
+          <mesh filename="package://turtlebot_description/meshes/stacks/circles/68-04552-1000-RA_Turtlebot_M-F_Standoff.dae"/>
         </geometry>
       </visual>
@@ -74,5 +74,5 @@
         <origin xyz=" 0 0 0 " rpy="0 0 0" />
         <geometry>
-          <mesh filename="package://gatlin/meshes/stacks/circles/68-04552-2000-RA_Turtlebot_M-F_Standoff.dae"/>
+          <mesh filename="package://turtlebot_description/meshes/stacks/circles/68-04552-2000-RA_Turtlebot_M-F_Standoff.dae"/>
         </geometry>
       </visual>
@@ -102,5 +102,5 @@
         <origin xyz=" 0 0 0 " rpy="0 0 0" />
         <geometry>
-          <mesh filename="package://gatlin/meshes/stacks/circles/68-02421-8000-RA_Turtlebot_F-F_Standoff.dae"/>
+          <mesh filename="package://turtlebot_description/meshes/stacks/circles/68-02421-8000-RA_Turtlebot_F-F_Standoff.dae"/>
         </geometry>
       </visual>
@@ -130,5 +130,5 @@
         <origin xyz=" 0 0 0 " rpy="0 0 0" />
         <geometry>
-          <mesh filename="package://gatlin/meshes/stacks/circles/68-04556-RA_Kinect_Standoff_Assy.dae"/>
+          <mesh filename="package://turtlebot_description/meshes/stacks/circles/68-04556-RA_Kinect_Standoff_Assy.dae"/>
         </geometry>
       </visual>
@@ -141,5 +141,5 @@
     </link>
   </xacro:macro>
-  <xacro:macro name="stack_circles" params="parent offset top_plate">
+  <xacro:macro name="stack_circles" params="parent">
     <turtlebot_spacer parent="${parent}" number="0" x_loc="-0.00254" y_loc="0.1114679" z_loc="0.062992"/>
     <turtlebot_spacer parent="${parent}" number="1" x_loc="-0.00254" y_loc="-0.1114679" z_loc="0.062992"/>
@@ -162,5 +162,5 @@
         <origin xyz=" 0 0 0 " rpy="0 0 0" />
         <geometry>
-          <mesh filename="package://gatlin/meshes/stacks/circles/plate_0_logo.dae"/>
+          <mesh filename="package://turtlebot_description/meshes/stacks/circles/plate_0_logo.dae"/>
         </geometry>
       </visual>
@@ -177,5 +177,5 @@
     <turtlebot_standoff_2in parent="${parent}" number="3" x_loc="-0.052832" y_loc="0.1314196" z_loc="0.0709803"/>
     <joint name="plate_1_joint" type="fixed">
-      <origin xyz="${0.04068+offset} 0 0.05715" rpy="0 0 0" />
+      <origin xyz="0.04068 0 0.05715" rpy="0 0 0" />
       <parent link="plate_0_link"/>
       <child link="plate_1_link" />
@@ -192,5 +192,5 @@
         <origin xyz=" 0 0 0 " rpy="0 0 0" />
         <geometry>
-          <mesh filename="package://gatlin/meshes/stacks/circles/plate_1_logo.dae"/>
+          <mesh filename="package://turtlebot_description/meshes/stacks/circles/plate_1_logo.dae"/>
         </geometry>
       </visual>
@@ -222,5 +222,5 @@
         <origin xyz=" 0 0 0 " rpy="0 0 0" />
         <geometry>
-          <mesh filename="package://gatlin/meshes/stacks/circles/plate_1_logo.dae"/>
+          <mesh filename="package://turtlebot_description/meshes/stacks/circles/plate_1_logo.dae"/>
         </geometry>
       </visual>
@@ -239,5 +239,5 @@
     <turtlebot_standoff_8in parent="standoff_2in_7_link" number="3" x_loc="0" y_loc="0" z_loc="0.05715"/>
     <joint name="plate_3_joint" type="fixed">
-      <origin xyz="-0.01316 0 ${0.2063496+top_plate}" rpy="0 0 0" />
+      <origin xyz="-0.01316 0 0.2063496" rpy="0 0 0" />
       <parent link="plate_2_link"/>
       <child link="plate_3_link" />
@@ -254,5 +254,5 @@
         <origin xyz=" 0 0 0 " rpy="0 0 0" />
         <geometry>
-          <mesh filename="package://gatlin/meshes/stacks/circles/plate_2_logo.dae"/>
+          <mesh filename="package://turtlebot_description/meshes/stacks/circles/plate_2_logo.dae"/>
         </geometry>
       </visual>

File: urdf/turtlebot_library.urdf.xacro (robot description, xacro)
@@ -9,11 +9,8 @@
   <!-- Bases -->
   <xacro:include filename="$(find gatlin)/urdf/create.urdf.xacro"/>
-  <!-- <xacro:include filename="$(find kobuki_description)/urdf/kobuki.urdf.xacro" /> -->
   <!-- Stacks -->
   <xacro:include filename="$(find gatlin)/urdf/stacks/circles.urdf.xacro"/>
   <xacro:include filename="$(find gatlin)/urdf/stacks/squares.urdf.xacro"/>
-  <!-- <xacro:include filename="$(find turtlebot_description)/urdf/stacks/hexagons.urdf.xacro"/> -->
   <!-- 3D Sensors -->
-  <!-- <xacro:include filename="$(find turtlebot_description)/urdf/sensors/kinect.urdf.xacro"/> -->
-  <!-- <xacro:include filename="$(find turtlebot_description)/urdf/sensors/asus_xtion_pro.urdf.xacro"/> -->
+  <xacro:include filename="$(find gatlin)/urdf/sensors/kinect.urdf.xacro"/>
 </robot>

Commit message: gatlin simulator kinect and gmapping working, arm and head servos not working

File: robots/gatlin_with_arm_and_head.urdf.xacro (robot description, xacro)
@@ -1,9 +1,8 @@
 <?xml version="1.0"?>
-<robot name="turtlebot" xmlns:xacro="http://ros.org/wiki/xacro">
-<!-- <robot name="gatlin_robot" xmlns:xacro="http://ros.org/wiki/xacro"> -->
+<robot name="gatlin_robot" xmlns:xacro="http://ros.org/wiki/xacro">
    <xacro:property name="PI" value="3.1415"/>
    <!-- Define a number of dimensions using properties -->
    <property name="head_offset_x" value="0.075" />
-   <property name="head_offset_y" value="0.02" />
+   <property name="head_offset_y" value="0.00" />
    <property name="head_offset_z" value="0.035" />
    <property name="head_offset_rotz" value="0.02" />
@@ -30,14 +29,12 @@
    <create/>
    <!-- Attach the stacks -->
-   <!-- <stack_circles parent="base_link"/> -->
    <stack_squares parent="base_link" offset="${stacks_offset}" top_plate="${top_plate}"/>
    <!-- Attach the pan and tilt head -->
-   <!-- <sensor_kinect  parent="base_link"/> -->
    <head name="head_base" parent="plate_3" color="White">
       <origin xyz="${head_offset_x} ${head_offset_y} ${head_offset_z}" rpy="${PI/2} 0 ${PI/2+head_offset_rotz}" />
    </head>
    <!-- Attach the arm -->
-   <!-- <turtlebot_arm parent="base_link" color="Gray" gripper_color="Gray" pincher_gripper="true" turtlebot_gripper="false">
+   <turtlebot_arm parent="base_link" color="Gray" gripper_color="Gray" pincher_gripper="true" turtlebot_gripper="false">
       <origin xyz="${arm_offset_x} ${arm_offset_y} ${arm_offset_z}" rpy="0 0 0" />
-   </turtlebot_arm> -->
+   </turtlebot_arm>
 </robot>

File: urdf/pan_tilt_head.urdf.xacro (robot description, xacro)
@@ -1,11 +1,11 @@
 <?xml version="1.0"?>
 <robot name="pan_tilt_head" xmlns:xacro="http://ros.org/wiki/xacro">
-  <property name="camera_offset_x" value="0.0" />
-  <property name="camera_offset_y" value="0.0" />
-  <property name="camera_offset_z" value="0.0615" />
+  <property name="camera_offset_x" value="0.02" />
+  <property name="camera_offset_y" value="-0.013" />
+  <property name="camera_offset_z" value="0.07" />
   <property name="camera_mesh_scale" value="1.0" />
   <xacro:include filename="$(find turtlebot_arm_description)/urdf/arm_hardware.xacro"/>
   <!-- <xacro:include filename="$(find gatlin)/urdf/dynamixel_head_hardware.xacro" /> -->
-  <xacro:include filename="$(find gatlin)/urdf/kinect.urdf.xacro" />
+  <xacro:include filename="$(find gatlin)/urdf/sensors/kinect.urdf.xacro" />
   <macro name="head" params="parent name color *origin">
     <!-- head base joint -->
@@ -50,8 +50,11 @@
        <origin xyz="0 0 0" rpy="0 0 0" />
     </bioloid_F2_revolute>
-   <!-- Attach the camera -->
-   <camera name="camera" parent="head_tilt" color="Black">
+    <!-- Attach the camera -->
+    <!-- <camera name="camera" parent="head_tilt" color="Black">
       <origin xyz="${camera_offset_x} ${camera_offset_y} ${camera_offset_z}" rpy="0 0 0" />
-   </camera>
- </macro>
+    </camera> -->
+    <sensor_kinect  parent="head_tilt_link" >
+      <origin xyz="${camera_offset_x} ${camera_offset_y} ${camera_offset_z}" rpy="0 0 0" />
+    </sensor_kinect>
+  </macro>
 </robot>

File: urdf/pincher_arm.urdf (robot description, URDF)
Before this commit: robot turtlebot_arm, 23 links, 23 joints
Links:
- removed link arm_base_link
- removed link arm_elbow_F10_0_link
- removed link arm_elbow_F10_1_link
- removed link arm_elbow_F10_2_link
- removed link arm_elbow_F3_0_link
- removed link arm_elbow_flex_link
- removed link arm_elbow_flex_servo_link
- removed link arm_shoulder_F10_0_link
- removed link arm_shoulder_F10_1_link
- removed link arm_shoulder_F10_2_link
- removed link arm_shoulder_F3_0_link
- removed link arm_shoulder_lift_link
- removed link arm_shoulder_lift_servo_link
- removed link arm_shoulder_pan_link
- removed link arm_shoulder_pan_servo_link
- removed link arm_wrist_F3_0_link
- removed link arm_wrist_flex_link
- removed link arm_wrist_flex_servo_link
- removed link gripper_active2_link
- removed link gripper_active_link
- removed link gripper_finger_base_link
- removed link gripper_link
- removed link gripper_servo_link
Joints:
- removed joint arm_base_joint
- removed joint arm_elbow_F10_0_joint
- removed joint arm_elbow_F10_1_joint
- removed joint arm_elbow_F10_2_joint
- removed joint arm_elbow_F3_0_joint
- removed joint arm_elbow_flex_joint
- removed joint arm_elbow_flex_servo_joint
- removed joint arm_shoulder_F10_0_joint
- removed joint arm_shoulder_F10_1_joint
- removed joint arm_shoulder_F10_2_joint
- removed joint arm_shoulder_F3_0_joint
- removed joint arm_shoulder_lift_joint
- removed joint arm_shoulder_lift_servo_joint
- removed joint arm_shoulder_pan_joint
- removed joint arm_shoulder_pan_servo_joint
- removed joint arm_wrist_F3_0_joint
- removed joint arm_wrist_flex_joint
- removed joint arm_wrist_flex_servo_joint
- removed joint gripper2_joint
- removed joint gripper_finger_base_joint
- removed joint gripper_joint
- removed joint gripper_link_joint
- removed joint gripper_servo_joint

File: urdf/sensors/kinect.urdf.xacro (robot description, xacro)
@@ -5,7 +5,8 @@
   <xacro:property name="kinect_cam_py" value="-0.0125"/>
   <!-- Parameterised in part by the values in turtlebot_properties.urdf.xacro -->
-  <xacro:macro name="sensor_kinect" params="parent">
+  <macro name="sensor_kinect" params="parent *origin">
     <joint name="camera_rgb_joint" type="fixed">
-      <origin xyz="${cam_px} ${kinect_cam_py} ${cam_pz}" rpy="${cam_or} ${cam_op} ${cam_oy}"/>
+      <insert_block name="origin"/>
+      <!-- <origin xyz=".02 0 0.0615" rpy="0 0 0"/> -->
       <parent link="${parent}"/>
       <child link="camera_rgb_frame" />
@@ -23,5 +24,5 @@
       <child link="camera_link"/>
     </joint>
-      <link name="camera_link">
+    <link name="camera_link">
       <visual>
        <origin xyz="0 0 0" rpy="0 0 ${M_PI/2}"/>
@@ -30,10 +31,10 @@
         </geometry>
       </visual>
-  	  <collision>
+      <collision>
         <origin xyz="0.0 0.0 0.0" rpy="0 0 0"/>
-  	    <geometry>
-  	      <box size="0.07271 0.27794 0.073"/>
-  	    </geometry>
-  	  </collision>
+        <geometry>
+          <box size="0.07271 0.27794 0.073"/>
+        </geometry>
+      </collision>
       <inertial>
         <mass value="0.564" />
@@ -47,18 +48,19 @@
          files. However, for Gazebo simulation we need them, so we add them here.
          (Hence, don't publish them additionally!) -->
-	<joint name="camera_depth_joint" type="fixed">
-	  <origin xyz="0 ${2 * -kinect_cam_py} 0" rpy="0 0 0" />
-	  <parent link="camera_rgb_frame" />
-	  <child link="camera_depth_frame" />
-	</joint>
-	<link name="camera_depth_frame"/>
-	<joint name="camera_depth_optical_joint" type="fixed">
-	  <origin xyz="0 0 0" rpy="${-M_PI/2} 0 ${-M_PI/2}" />
-	  <parent link="camera_depth_frame" />
-	  <child link="camera_depth_optical_frame" />
-	</joint>
-	<link name="camera_depth_optical_frame"/>
-	<!-- Kinect sensor for simulation -->
-	<turtlebot_sim_3dsensor/>
-  </xacro:macro>
+    <joint name="camera_depth_joint" type="fixed">
+      <origin xyz="0 ${2 * -kinect_cam_py} 0" rpy="0 0 0" />
+      <parent link="camera_rgb_frame" />
+      <child link="camera_depth_frame" />
+    </joint>
+    <link name="camera_depth_frame"/>
+    <joint name="camera_depth_optical_joint" type="fixed">
+      <origin xyz="0 0 0" rpy="${-M_PI/2} 0 ${-M_PI/2}" />
+      <parent link="camera_depth_frame" />
+      <child link="camera_depth_optical_frame" />
+    </joint>
+    <link name="camera_depth_optical_frame"/>
+    <!-- Kinect sensor for simulation -->
+    <turtlebot_sim_3dsensor/>
+    <!-- causing problems for some reason -->
+  </macro>
 </robot>

File: urdf/turtlebot_gazebo.urdf.xacro (robot description, xacro)
@@ -6,5 +6,5 @@
       <sensor type="depth" name="camera">
         <always_on>true</always_on>
-        <update_rate>20.0</update_rate>
+        <update_rate>30.0</update_rate>
         <camera>
           <horizontal_fov>${60.0*M_PI/180.0}</horizontal_fov>
