Commit message: added Multi Robot sim, not working yet with tf_prefix on fake kinect

File: robots/create_circles_kinect.urdf.xacro (robot description, xacro)
@@ -9,4 +9,6 @@
   <create/>
   <stack_circles parent="base_link"/>
-  <sensor_kinect  parent="base_link"/>
+  <sensor_kinect  parent="base_link" >
+    <origin xyz="${cam_px} 0 ${cam_pz}" rpy="0 0 0" />
+  </sensor_kinect>
 </robot>

Commit message: added plannar laser scan

File: robots/create_circles_kinect.urdf.xacro (robot description, xacro)
@@ -10,5 +10,6 @@
   <stack_circles parent="base_link"/>
   <sensor_kinect  parent="base_link" >
-    <origin xyz="${cam_px} 0 ${cam_pz}" rpy="0 0 0" />
+    <!-- <origin xyz="${cam_px} 0 ${cam_pz}" rpy="0 0 0" /> -->
+    <origin xyz="${cam_px} 0 .6" rpy="0 .4 0" />
   </sensor_kinect>
 </robot>
