Commit message: still trying to get gatlin sim working

File: urdf/create.urdf.xacro (robot description, xacro)
@@ -188,6 +188,6 @@
 	  </link>
 	  <!-- fixed because there's no transmission -->
-	  <!-- <joint name="rear_castor_joint" type="fixed"> -->
-	  <joint name="back_castor_joint" type="fixed">
+	  <joint name="rear_castor_joint" type="fixed">
+	  <!-- <joint name="back_castor_joint" type="fixed"> -->
 	    <origin xyz="-0.129 0 0.0" rpy="0 0 0"/>
 	    <parent link="base_link"/>

File: urdf/create_gazebo.urdf.xacro (robot description, xacro)
@@ -9,5 +9,6 @@
 	      <right_wheel_joint>right_wheel_joint</right_wheel_joint>
 	      <front_castor_joint>front_castor_joint</front_castor_joint>
-	      <rear_castor_joint>rear_castor_joint</rear_castor_joint>
+        <rear_castor_joint>rear_castor_joint</rear_castor_joint>
+	      <!-- <back_castor_joint>back_castor_joint</back_castor_joint> -->
 	      <wheel_separation>.260</wheel_separation>
 	      <wheel_diameter>0.066</wheel_diameter>
